Commit message: Rotate gripper model for visualization

File: final_project/src/universal_robot/ur_description/urdf/ur.xacro (robot description, xacro)
@@ -31,5 +31,5 @@
    <xacro:robotiq_arg2f_140 prefix=""/>
       <joint name='ur5_to_gripper_joint' type="fixed">
-         <origin xyz="0 0 0.1" rpy="0 0 0"/>
+         <origin xyz="0 0 0.1" rpy="0 0 ${pi / 2 }"/>
          <parent link="tool0"/>
          <child link="robotiq_arg2f_base_link"/>
