Commit message: Add gripper and collision geometry to UR5 robot

File: final_project/src/robotiq/robotiq_2f_140_gripper_visualization/urdf/robotiq_arg2f.xacro (robot description, xacro)
@@ -18,8 +18,8 @@
       </visual>
       <collision>
-        <origin xyz="0 0 0" rpy="0 0 0" />
-        <geometry>
-          <mesh filename="package://robotiq_2f_140_gripper_visualization/meshes/collision/robotiq_arg2f_base_link.stl" />
-        </geometry>
+            <origin xyz="0 0 0.11" rpy="0 0 0" />
+            <geometry>
+            <cylinder length="0.22" radius="0.15"/>
+            </geometry>
       </collision>
     </link>

File: final_project/src/robotiq/robotiq_2f_140_gripper_visualization/urdf/robotiq_arg2f_140_model_macro.xacro (robot description, xacro)
@@ -24,10 +24,4 @@
         </material>
       </visual>
-      <collision>
-        <origin xyz="0 0 0" rpy="0 0 0" />
-        <geometry>
-          <mesh filename="package://robotiq_2f_140_gripper_visualization/meshes/collision/robotiq_arg2f_${stroke}_outer_knuckle.stl" />
-        </geometry>
-      </collision>
     </link>
   </xacro:macro>
@@ -54,10 +48,4 @@
         </material>
       </visual>
-      <collision>
-        <origin xyz="0 0 0" rpy="0 0 0" />
-        <geometry>
-          <mesh filename="package://robotiq_2f_140_gripper_visualization/meshes/collision/robotiq_arg2f_${stroke}_outer_finger.stl" />
-        </geometry>
-      </collision>
     </link>
   </xacro:macro>
@@ -84,10 +72,4 @@
         </material>
       </visual>
-      <collision>
-        <origin xyz="0 0 0" rpy="0 0 0" />
-        <geometry>
-          <mesh filename="package://robotiq_2f_140_gripper_visualization/meshes/collision/robotiq_arg2f_${stroke}_inner_knuckle.stl" />
-        </geometry>
-      </collision>
     </link>
   </xacro:macro>
@@ -114,10 +96,4 @@
         </material>
       </visual>
-      <collision>
-        <origin xyz="0 0 0" rpy="0 0 0" />
-        <geometry>
-          <mesh filename="package://robotiq_2f_140_gripper_visualization/meshes/collision/robotiq_arg2f_${stroke}_inner_finger.stl" />
-        </geometry>
-      </collision>
     </link>
   </xacro:macro>
@@ -134,13 +110,4 @@
         </material>
       </visual>
-      <collision>
-        <origin xyz="0 0 0" rpy="0 0 0" />
-        <geometry>
-           <box size="0.03 0.07 0.0075"/>
-        </geometry>
-        <material name="">
-          <color rgba="0.9 0.0 0.0 1" />
-        </material>
-      </collision>
     </link>
   </xacro:macro>

File: final_project/src/universal_robot/ur_description/urdf/ur.xacro (robot description, xacro)
@@ -3,4 +3,5 @@
    <!-- import main macro -->
    <xacro:include filename="$(find ur_description)/urdf/inc/ur_macro.xacro"/>
+   <xacro:include filename="$(find robotiq_2f_140_gripper_visualization)/urdf/robotiq_arg2f_140_model_macro.xacro" />
    <!-- parameters -->
    <xacro:arg name="joint_limit_params" default=""/>
@@ -28,3 +29,9 @@
      safety_pos_margin="$(arg safety_pos_margin)"
      safety_k_position="$(arg safety_k_position)"/>
+   <xacro:robotiq_arg2f_140 prefix=""/>
+      <joint name='ur5_to_gripper_joint' type="fixed">
+         <origin xyz="0 0 0.1" rpy="0 0 0"/>
+         <parent link="tool0"/>
+         <child link="robotiq_arg2f_base_link"/>
+      </joint>
 </robot>

Commit message: Better collision boxes

File: final_project/src/robotiq/robotiq_2f_140_gripper_visualization/urdf/robotiq_arg2f.xacro (robot description, xacro)
@@ -18,7 +18,7 @@
       </visual>
       <collision>
-            <origin xyz="0 0 0.11" rpy="0 0 0" />
+            <origin xyz="0 0 0.088" rpy="0 0 0" />
             <geometry>
-            <cylinder length="0.22" radius="0.15"/>
+            <cylinder length="0.3048" radius="0.1"/>
             </geometry>
       </collision>

File: final_project/src/universal_robot/ur_description/urdf/ur.xacro (robot description, xacro)
@@ -31,5 +31,5 @@
    <xacro:robotiq_arg2f_140 prefix=""/>
       <joint name='ur5_to_gripper_joint' type="fixed">
-         <origin xyz="0 0 0.1" rpy="0 0 ${pi / 2 }"/>
+         <origin xyz="0 0 0.0650875" rpy="0 0 ${pi / 2 }"/>
          <parent link="tool0"/>
          <child link="robotiq_arg2f_base_link"/>
